Commit message: fix urdf astracam

File: src/tirocinio/urdf/turtlebot3_burger_camera.urdf.xacro (robot description, xacro)
@@ -101,5 +101,5 @@
     <parent link="base_link"/>
     <child link="camera_link"/>
-    <origin rpy="0.0062 0.7527 0" xyz="0.09 0.06 1.5737"/>             # TODO calibrate
+    <origin rpy="0 0 0" xyz="0.05 0.06 0.15"/>
   </joint>
   <joint name="caster_back_joint" type="fixed">

Commit message: settata nuova camera e ""calibrata""

File: src/tirocinio/urdf/turtlebot3_burger_camera.urdf.xacro (robot description, xacro)
@@ -95,5 +95,5 @@
       </geometry>
       <material name="black"/>
-      <origin rpy="0 0 0" xyz="0 -0.06 0.0"/>     # Displacement/Rotation of the center with respect camera_up_link
+      <origin rpy="0 0 0" xyz="-0.10 -0.06 0.15"/>     # Displacement/Rotation of the center with respect camera_up_link
     </visual>
   </link>
@@ -101,5 +101,5 @@
     <parent link="base_link"/>
     <child link="camera_link"/>
-    <origin rpy="0 0 0" xyz="0.05 0.06 0.15"/>
+    <origin rpy="0 0.23 0" xyz="0.05 0.06 0.30"/>
   </joint>
   <joint name="caster_back_joint" type="fixed">
